File: Controller KiCad/Controller.kicad_sch (KiCad schematic)
At the start: 11 parts, among them J1 ESP32 L-Header, J2 ESP32 R-Header, J3 Conn_01x05, SW1 SW_Push, SW2 SW_Push, SW3 SW_Push, SW4 SW_Push

Commit message: Finished schematic
Connections:
- net +3V3: now also R1.1, R2.1, R3.1, R4.1, SW1.1, SW2.1, SW3.1, SW4.1
- net SW: no longer names the net of J3.5 (Pin_5)
- no-connect marks 42 -> 22
Other:
- title: (none) -> Controller
- moved on the sheet: J1, J2, J3

Commit message: Almost complete PCB
Parts:
- J1, J2: footprint (none) -> Connector_PinHeader_2.54mm:PinHeader_1x15_P2.54mm_Vertical
- J3: footprint (none) -> Connector_PinHeader_2.54mm:PinHeader_1x05_P2.54mm_Vertical
- R1, R2, R3, R4: footprint (none) -> Resistor_THT:R_Axial_DIN0207_L6.3mm_D2.5mm_P7.62mm_Horizontal
- SW1, SW2, SW3, SW4: footprint (none) -> Button_Switch_THT:SW_PUSH_6mm
