File: Controller KiCad/_restore_backup_2026-10-07T21-09-07-048/Controller.kicad_pcb (KiCad board)
At the start: 2 copper layers, 130 x 73 mm, 17 parts, among them J1 ESP32 L-Header, J2 ESP32 R-Header, J3 Conn_01x05, SW1 SW_Push, SW2 SW_Push, SW3 SW_Push, SW4 SW_Push

Commit message: Slight updates that took a long time
Parts:
- removed D1: LED, LED_THT:LED_D5.0mm
- removed H1, H2, H3, H4: 4.0mm, MountingHole:MountingHole_4mm
- removed R5: 330, Resistor_THT:R_Axial_DIN0207_L6.3mm_D2.5mm_P7.62mm_Horizontal
- added REF**: MountingHole_3.2mm, MountingHole:MountingHole_2.1mm, F.Cu at (80.0, 47.6)
- added REF**: MountingHole_3.2mm, MountingHole:MountingHole_2.1mm, F.Cu at (80.0, 73.6)
- added REF**: MountingHole_3.2mm, MountingHole:MountingHole_2.1mm, F.Cu at (60.0, 73.6)
- added REF**: MountingHole_3.2mm, MountingHole:MountingHole_2.1mm, F.Cu at (60.0, 47.6)
- moved J3 21.3 mm to (107.8, 114.4)
Other:
- board outline removed
