File: Controller KiCad/_restore_backup_2026-10-07T21-09-07-048/Controller.kicad_sch (KiCad schematic)
At the start: 17 parts, among them J1 ESP32 L-Header, J2 ESP32 R-Header, J3 Conn_01x05, SW1 SW_Push, SW2 SW_Push, SW3 SW_Push, SW4 SW_Push

Commit message: Slight updates that took a long time
Parts:
- removed D1: LED, LED_THT:LED_D5.0mm, symbol Device:LED
- removed H1, H2, H3, H4: 4.0mm, MountingHole:MountingHole_4mm, symbol Mechanical:MountingHole
- removed R5: 330, Resistor_THT:R_Axial_DIN0207_L6.3mm_D2.5mm_P7.62mm_Horizontal, symbol Device:R
Connections:
- no-connect marks 21 -> 22
